File: test-rc/2x-rc.kicad_pcb (KiCad board)
At the start: 2 copper layers, 6 parts, among them J1 CONN_01X02, J2 CONN_01X02

Commit message: add readme with screenshots
Parts:
- moved J2 21.5 mm to (141.6, 111.1), turned to 180 degrees
- moved J1 18.5 mm to (154.9, 111.1), turned to 180 degrees
- moved R1 10.8 mm to (148.8, 112.5)
- moved R2 10.8 mm to (148.9, 115.8)
- moved C1 10.8 mm to (149.0, 105.4)
- moved C2 10.8 mm to (149.5, 108.3)
Changed lines of the file:
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@@
     (links 7)
     (no_connects 7)
-    (area 0 0 0 0)
+    (area 137.968667 102.97 161.497334 119.6086)
     (thickness 1.6)
     (drawings 0)
@@
   )
   (module Capacitors_SMD:C_0805_HandSoldering (layer F.Cu)
-    (at 149.225 94.615)
+    (at 148.971 105.41)
     (descr "Capacitor SMD 0805, hand soldering")
     (tags "capacitor 0805")
@@
   )
   (module Capacitors_SMD:C_0805_HandSoldering (layer F.Cu)
-    (at 149.733 97.536)
+    (at 149.479 108.331)
     (descr "Capacitor SMD 0805, hand soldering")
     (tags "capacitor 0805")
@@
   )
   (module Pin_Headers:Pin_Header_Straight_1x02 (layer F.Cu)
-    (at 166.878 97.028)
+    (at 154.94 111.125 180)
     (descr "Through hole pin header")
     (tags "pin header")
-    (fp_text reference J1 (at 0 -5.1) (layer F.SilkS)
-      (effects (font (size 1 1) (thickness 0.15)))
-    )
-    (fp_text value CONN_01X02 (at 0 -3.1) (layer F.Fab)
+    (fp_text reference J1 (at 0 -5.1 180) (layer F.SilkS)
+      (effects (font (size 1 1) (thickness 0.15)))
+    )
+    (fp_text value CONN_01X02 (at 0 -3.1 180) (layer F.Fab)
       (effects (font (size 1 1) (thickness 0.15)))
     )
@@
     (fp_line (start -1.27 1.27) (end -1.27 3.81) (layer F.SilkS) (width 0.15))
     (fp_line (start -1.27 3.81) (end 1.27 3.81) (layer F.SilkS) (width 0.15))
-    (pad 1 thru_hole rect (at 0 0) (size 2.032 2.032) (drill 1.016) (layers *.Cu *.Mask F.SilkS)
+    (pad 1 thru_hole rect (at 0 0 180) (size 2.032 2.032) (drill 1.016) (layers *.Cu *.Mask F.SilkS)
       (net 3 /rc/In))
-    (pad 2 thru_hole oval (at 0 2.54) (size 2.032 2.032) (drill 1.016) (layers *.Cu *.Mask F.SilkS)
+    (pad 2 thru_hole oval (at 0 2.54 180) (size 2.032 2.032) (drill 1.016) (layers *.Cu *.Mask F.SilkS)
       (net 4 /rc2/In))
     (model Pin_Headers.3dshapes/Pin_Header_Straight_1x02.wrl
@@
   )
   (module Pin_Headers:Pin_Header_Straight_1x02 (layer F.Cu)
-    (at 130.429 92.71)
+    (at 141.605 111.125 180)
     (descr "Through hole pin header")
     (tags "pin header")
-    (fp_text reference J2 (at 0 -5.1) (layer F.SilkS)
-      (effects (font (size 1 1) (thickness 0.15)))
-    )
-    (fp_text value CONN_01X02 (at 0 -3.1) (layer F.Fab)
+    (fp_text reference J2 (at 0 -5.1 180) (layer F.SilkS)
+      (effects (font (size 1 1) (thickness 0.15)))
+    )
+    (fp_text value CONN_01X02 (at 0 -3.1 180) (layer F.Fab)
       (effects (font (size 1 1) (thickness 0.15)))
     )
@@
     (fp_line (start -1.27 1.27) (end -1.27 3.81) (layer F.SilkS) (width 0.15))
     (fp_line (start -1.27 3.81) (end 1.27 3.81) (layer F.SilkS) (width 0.15))
-    (pad 1 thru_hole rect (at 0 0) (size 2.032 2.032) (drill 1.016) (layers *.Cu *.Mask F.SilkS)
+    (pad 1 thru_hole rect (at 0 0 180) (size 2.032 2.032) (drill 1.016) (layers *.Cu *.Mask F.SilkS)
       (net 1 /rc/Out))
-    (pad 2 thru_hole oval (at 0 2.54) (size 2.032 2.032) (drill 1.016) (layers *.Cu *.Mask F.SilkS)
+    (pad 2 thru_hole oval (at 0 2.54 180) (size 2.032 2.032) (drill 1.016) (layers *.Cu *.Mask F.SilkS)
       (net 2 /rc2/Out))
     (model Pin_Headers.3dshapes/Pin_Header_Straight_1x02.wrl
@@
   )
   (module Resistors_SMD:R_0805_HandSoldering (layer F.Cu)
-    (at 148.463 101.727)
+    (at 148.844 112.522)
     (descr "Resistor SMD 0805, hand soldering")
     (tags "resistor 0805")
@@
   )
   (module Resistors_SMD:R_0805_HandSoldering (layer F.Cu)
-    (at 148.5011 105.0036)
+    (at 148.8821 115.7986)
     (descr "Resistor SMD 0805, hand soldering")
     (tags "resistor 0805")
